File: Tympan_D.kicad_pcb (KiCad board)
At the start: 4 copper layers, 38 x 74 mm, 116 parts, among them IC1 MK66FX1M0VMD18, IC2 MKL02Z32VFG4, IC3 BC127, J1 SJ-3523-SMT-TR, J2 SJ-3524-SMT-TR-PI, J3 alt Power Pads, P1 USB_OTG, P10 CONN_01X01, P2 CONN_01X06, P3 CONN_01X06, P4 CONN_01X06, P5 CONN_01X06, P6 CONN_01X03, P7 CONN_01X01, P8 CONN_01X01, P9 CONN_01X01, SW1 CL-SB-22A, SW2 TACT_SWITCH, U1 AP2210K-3.3TRG1, U2 TLV320AIC3206IRSBT, U3 74LVC1G66, U4 LP5907MFX-1.8, U5 MCP73831, Y1 32.768kHz, Y2 16MHz

Commit message: Changed the silks, changed rev before my changes applied.
Other:
- board text added: "Designed in Brooklyn, NY USA"
- board text added: "TYMPAN Rev D_SB"
- board text added: "TYMPAN RevD_SB"
- board text removed: "Designed in Brooklyn, NY USA Made in Taipei, Taiwan"
- board text removed: "TYMPAN Rev D"
- board text removed: "TYMPAN RevD"
Changed lines of the file:
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@@
-(kicad_pcb (version 20171130) (host pcbnew "(5.0.1-3-g963ef8bb5)")
+(kicad_pcb (version 20171130) (host pcbnew 5.1.1-8be2ce7~80~ubuntu18.04.1)
   (general
     (thickness 1.6)
@@
     (38 B.Mask user)
     (39 F.Mask user)
-    (40 Dwgs.User user)
+    (40 Dwgs.User user hide)
     (41 Cmts.User user hide)
     (42 Eco1.User user hide)
-    (43 Eco2.User user)
+    (43 Eco2.User user hide)
     (44 Edge.Cuts user)
-    (45 Margin user)
-    (46 B.CrtYd user)
-    (47 F.CrtYd user)
+    (45 Margin user hide)
+    (46 B.CrtYd user hide)
+    (47 F.CrtYd user hide)
     (48 B.Fab user hide)
     (49 F.Fab user hide)
@@
     (zone_45_only yes)
     (trace_min 0.1778)
-    (segment_width 0.2)
-    (edge_width 0.15)
     (via_size 0.6)
     (via_drill 0.4)
@@
     (uvia_min_size 0.2)
     (uvia_min_drill 0.1)
+    (edge_width 0.15)
+    (segment_width 0.2)
     (pcb_text_width 0.2)
     (pcb_text_size 1 1)
@@
     (tags "capacitor 0402")
     (attr smd)
-    (fp_text reference C41 (at 0.06 -0.9) (layer F.SilkS)
+    (fp_text reference C41 (at 1.9206 0.0384) (layer F.SilkS)
       (effects (font (size 0.635 0.635) (thickness 0.127)))
     )
@@
     (effects (font (size 1 1) (thickness 0.2)) (justify mirror))
   )
-  (gr_text "www.tympan.org\ngithub.com/tympan" (at 133.95 73.08) (layer B.SilkS)
+  (gr_text "www.tympan.org\ngithub.com/tympan" (at 134.0016 71.8898) (layer B.SilkS)
     (effects (font (size 1 1) (thickness 0.2)) (justify mirror))
   )
-  (gr_text "Designed in Brooklyn, NY USA\nMade in Taipei, Taiwan" (at 133.85 54.08) (layer B.SilkS)
+  (gr_text "Designed in Brooklyn, NY USA" (at 133.85 54.08) (layer B.SilkS)
     (effects (font (size 1 1) (thickness 0.2)) (justify mirror))
   )
@@
   (gr_line (start 149.85 101.23) (end 149.85 63.23) (angle 90) (layer Eco1.User) (width 0.2))
   (gr_line (start 119.85 101.23) (end 149.85 101.23) (angle 90) (layer Eco1.User) (width 0.2))
-  (gr_text "TYMPAN\nRevD" (at 132.54 107.89) (layer F.SilkS)
+  (gr_text "TYMPAN\nRevD_SB" (at 133.8238 106.9672) (layer F.SilkS)
     (effects (font (size 1.524 1.524) (thickness 0.2)) (justify right))
   )
-  (gr_text "TYMPAN  Rev D" (at 133.85 58.28) (layer B.SilkS)
+  (gr_text "TYMPAN  Rev D_SB" (at 133.4682 59.2152) (layer B.SilkS)
     (effects (font (size 1.524 1.524) (thickness 0.25)) (justify mirror))
   )
